File: Low-Ammo Detector/RingBoard/hopperBoard.sch (EAGLE design)
At the start: 17 parts

Commit message: added changes since repo changes
Parts:
- U$6: value XT30PW-M -> SM02B-GHS-TB; device _HenrySilva:XT30PW-M -> _HenrySilva:SM02B-GHS-TB
Connections:
- net 5V: now also U$6.1; no longer U$6.VCC
- net GND: now also U$6.2; no longer U$6.GND
Changed lines of the file:
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@@
 <part name="U$11" library="microbuilder" deviceset="MOUNTINGHOLE" device="3.0THIN"/>
 <part name="U$12" library="microbuilder" deviceset="MOUNTINGHOLE" device="3.0THIN"/>
-<part name="U$6" library="_HenrySilva" deviceset="XT30PW-M" device=""/>
 <part name="U$7" library="microbuilder" deviceset="MOUNTINGHOLE" device="3.0THIN"/>
+<part name="U$6" library="_HenrySilva" deviceset="SM02B-GHS-TB" device=""/>
 </parts>
 <sheets>
@@
 <instance part="U$11" gate="G$1" x="25.4" y="20.32" smashed="yes"/>
 <instance part="U$12" gate="G$1" x="43.18" y="20.32" smashed="yes"/>
-<instance part="U$6" gate="G$1" x="-45.72" y="63.5" smashed="yes" rot="R270"/>
 <instance part="U$7" gate="G$1" x="25.4" y="2.54" smashed="yes"/>
+<instance part="U$6" gate="G$1" x="-38.1" y="55.88" smashed="yes" rot="R90"/>
 </instances>
 <busses>
@@
 <wire x1="-12.7" y1="50.8" x2="-12.7" y2="45.72" width="0.1524" layer="91"/>
 <label x="-12.7" y="45.72" size="1.778" layer="95" rot="R270"/>
-</segment>
-<segment>
-<wire x1="-40.64" y1="50.8" x2="-40.64" y2="45.72" width="0.1524" layer="91"/>
-<label x="-40.64" y="45.72" size="1.778" layer="95" rot="R270"/>
-<pinref part="U$6" gate="G$1" pin="GND"/>
 </segment>
 <segment>
@@
 <label x="162.56" y="-5.08" size="1.778" layer="95" rot="R270"/>
 </segment>
+<segment>
+<pinref part="U$6" gate="G$1" pin="2"/>
+<wire x1="-43.18" y1="50.8" x2="-43.18" y2="45.72" width="0.1524" layer="91"/>
+<label x="-43.18" y="45.72" size="1.778" layer="95" rot="R270"/>
+</segment>
 </net>
 <net name="5V" class="0">
-<segment>
-<wire x1="-43.18" y1="50.8" x2="-43.18" y2="45.72" width="0.1524" layer="91"/>
-<label x="-43.18" y="45.72" size="1.778" layer="95" rot="R270"/>
-<pinref part="U$6" gate="G$1" pin="VCC"/>
-</segment>
 <segment>
 <pinref part="U$4" gate="G$1" pin="VCC"/>
@@
 <label x="104.14" y="25.4" size="1.778" layer="95" rot="R180"/>
 </segment>
+<segment>
+<pinref part="U$6" gate="G$1" pin="1"/>
+<wire x1="-40.64" y1="50.8" x2="-40.64" y2="45.72" width="0.1524" layer="91"/>
+<label x="-40.64" y="45.72" size="1.778" layer="95" rot="R270"/>
+</segment>
 </net>
