File: Low-Ammo Detector/RingBoard/hopperBoard.brd (EAGLE design)
At the start: 172.2 x 172.3 mm, 17 parts

Commit message: added changes since repo changes
Parts:
- U$6: value XT30PW-M -> SM02B-GHS-TB; device _HenrySilva:XT30 -> _HenrySilva:SM02B-GHS-TB
- moved U$6 11.1 mm to (77.0, -24.0), turned to 90 degrees
Connections:
- net 5V: now also U$6.P$3; no longer U$6.P$1
- net GND: now also U$6.P$4; no longer U$6.P$2
Routing:
- net 5V: track 1.26 -> 3.21 mm, vias 7 -> 8
Changed lines of the file:
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@@
 <setting verticaltext="up"/>
 </settings>
-<grid distance="1" unitdist="mm" unit="mm" style="lines" multiple="1" display="yes" altdistance="5" altunitdist="mil" altunit="mil"/>
+<grid distance="3.93700787" unitdist="mil" unit="mil" style="lines" multiple="1" display="yes" altdistance="5" altunitdist="mil" altunit="mil"/>
 <layers>
 <layer number="1" name="Top" color="4" fill="1" visible="yes" active="yes"/>
@@
 <layer number="27" name="tValues" color="7" fill="1" visible="yes" active="yes"/>
 <layer number="28" name="bValues" color="7" fill="1" visible="yes" active="yes"/>
-<layer number="29" name="tStop" color="7" fill="3" visible="no" active="yes"/>
+<layer number="29" name="tStop" color="7" fill="3" visible="yes" active="yes"/>
 <layer number="30" name="bStop" color="7" fill="6" visible="no" active="yes"/>
 <layer number="31" name="tCream" color="7" fill="4" visible="no" active="yes"/>
@@
 <param name="mlMinCreamFrame" value="0mil"/>
 <param name="mlMaxCreamFrame" value="0mil"/>
-<param name="mlViaStopLimit" value="0mil"/>
+<param name="mlViaStopLimit" value="22mil"/>
 <param name="srRoundness" value="0"/>
 <param name="srMinRoundness" value="0mil"/>
@@
 <element name="U$11" library="microbuilder" package="MOUNTINGHOLE_3.0_PLATEDTHIN" value="MOUNTINGHOLE3.0THIN" x="-54.841" y="-54.806" smashed="yes"/>
 <element name="U$12" library="microbuilder" package="MOUNTINGHOLE_3.0_PLATEDTHIN" value="MOUNTINGHOLE3.0THIN" x="-54.809" y="54.809" smashed="yes"/>
-<element name="U$6" library="_HenrySilva" package="XT30" value="XT30PW-M" x="70.5" y="-15" smashed="yes" rot="R270"/>
 <element name="U$7" library="microbuilder" package="MOUNTINGHOLE_3.0_PLATEDTHIN" value="MOUNTINGHOLE3.0THIN" x="54.764" y="54.872" smashed="yes"/>
+<element name="U$6" library="_HenrySilva" package="SM02B-GHS-TB" value="SM02B-GHS-TB" x="77" y="-24" smashed="yes" rot="R90"/>
 </elements>
 <signals>
@@
 <contactref element="C3" pad="2"/>
 <contactref element="R2" pad="1"/>
-<polygon width="0.25" layer="1" isolate="0.254" rank="2">
+<polygon width="0.254" layer="1" isolate="0.254" rank="2">
 <vertex x="0" y="88"/>
 <vertex x="88" y="88"/>
@@
 <vertex x="-88" y="88"/>
 </polygon>
-<contactref element="U$6" pad="P$2"/>
+<contactref element="U$6" pad="P$4"/>
 </signal>
 <signal name="5V">
@@
 <via x="74.93" y="-5.588" extent="1-16" drill="0.35"/>
 <wire x1="74.93" y1="-5.588" x2="74.164" y2="-4.5904" width="0.2032" layer="1"/>
-<contactref element="U$6" pad="P$1"/>
+<contactref element="U$6" pad="P$3"/>
+<wire x1="72.45" y1="-22.15" x2="70.5" y2="-22.1" width="0.508" layer="1"/>
+<via x="70.5" y="-22.1" extent="1-16" drill="0.55"/>
 </signal>
 <signal name="AMMO2">

Commit message: Ammo Board V2
Parts:
- R1: value 540k -> 330k
- R2: value 360k -> 180k
Changed lines of the file:
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@@
 </layers>
 <board>
-<fusionsync huburn="a.YnVzaW5lc3M6cHVyZHVlMjIy" projecturn="a.YnVzaW5lc3M6cHVyZHVlMjIyIzIwMTkxMTA4MjM1OTg1Nzgx" f3durn="urn:adsk.wipprod:dm.lineage:DUGREdU3ThqPfMAjgLCw6w" pcbguid="18e90121-f44a-4ee8-9cac-4a6ccbb78db5" lastpulledtime="" lastsyncedchangeguid="175dc6bc-0ef5-d30d-e000-40e42407e41a"/>
+<fusionsync huburn="a.YnVzaW5lc3M6cHVyZHVlMjIy" projecturn="a.YnVzaW5lc3M6cHVyZHVlMjIyIzIwMTkxMTA4MjM1OTg1Nzgx" f3durn="urn:adsk.wipprod:dm.lineage:DUGREdU3ThqPfMAjgLCw6w" pcbguid="18e90121-f44a-4ee8-9cac-4a6ccbb78db5" lastpulledtime="" lastsyncedchangeguid="3ecf64a5-fef9-4233-5cdc-7bf6968c843e"/>
 <plain>
 <wire x1="30.29038125" y1="80.62796875" x2="22.8865" y2="83.033640625" width="0.001" layer="20" curve="-103.69"/>
@@
 <attribute name="VALUE" x="77.369" y="1.6746" size="1.27" layer="27" rot="R90"/>
 </element>
-<element name="R1" library="rcl" library_urn="urn:adsk.eagle:library:334" package="R0603" package3d_urn="urn:adsk.eagle:package:23555/3" value="540k" x="77.964" y="-1.1904" smashed="yes" rot="R90">
+<element name="R1" library="rcl" library_urn="urn:adsk.eagle:library:334" package="R0603" package3d_urn="urn:adsk.eagle:package:23555/3" value="330k" x="77.964" y="-1.1904" smashed="yes" rot="R90">
 <attribute name="NAME" x="77.329" y="-1.8254" size="1.27" layer="25" rot="R90"/>
 <attribute name="POPULARITY" value="77" x="77.964" y="-1.1904" size="1.778" layer="27" font="vector" rot="R90" display="off"/>
@@
 <attribute name="VALUE" x="79.869" y="-1.8254" size="1.27" layer="27" rot="R90"/>
 </element>
-<element name="R2" library="rcl" library_urn="urn:adsk.eagle:library:334" package="R0603" package3d_urn="urn:adsk.eagle:package:23555/3" value="360k" x="77.964" y="-4.6904" smashed="yes" rot="R90">
+<element name="R2" library="rcl" library_urn="urn:adsk.eagle:library:334" package="R0603" package3d_urn="urn:adsk.eagle:package:23555/3" value="180k" x="77.964" y="-4.6904" smashed="yes" rot="R90">
 <attribute name="NAME" x="77.329" y="-5.3254" size="1.27" layer="25" rot="R90"/>
 <attribute name="POPULARITY" value="77" x="77.964" y="-4.6904" size="1.778" layer="27" font="vector" rot="R90" display="off"/>
