File: Heads-Up-Display-ToF/OledBoard/OledBoardSchematicV1.brd (EAGLE design)
At the start: 56.6 x 33.3 mm, 46 parts, among them U1 AP3012, U2 UG-2856KLBAG01_4WSPI, U3 ATMEGA328P_TQFP, U4 CH340C

Commit message: added changes that were left behind
Parts:
- U$5: value SM04B-GHS-TB -> SM03B-GHS-TB; device oledBoard:SM04B-GHS-TB -> oledBoard:SM03B-GHS-TB
- moved U$5 7.44 mm to (45.2, 16.3)
Connections:
- net AMMO1: now also U$5.P$4; no longer U$5.4
- net AMMO2: now also U$5.P$3; no longer U$5.3
- net AMMO3: no longer U$5.2
- net GND: now also U$5.P$5; no longer U$5.1
Routing:
- net AMMO3: track 7.16 -> 0.00 mm
- net AMMO1: track 8.74 -> 8.15 mm
- net AMMO2: track 7.35 -> 6.75 mm
Other:
- board text added: "CS"
- board text added: "MOSI"
- board text added: "VCC"
Changed lines of the file:
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@@
 <rectangle x1="11.15695" y1="16.40205" x2="18.82775" y2="16.41475" layer="22"/>
 <rectangle x1="11.23315" y1="16.41475" x2="18.75155" y2="16.42745" layer="22"/>
+<text x="26.9367" y="6.9596" size="0.8128" layer="25">CS</text>
+<text x="28.9433" y="0.3937" size="0.8128" layer="25">MOSI</text>
+<text x="26.0985" y="0.4826" size="0.8128" layer="25">GND</text>
+<text x="32.512" y="0.3683" size="0.8128" layer="25">VCC</text>
 </plain>
 <attributes>
@@
 <element name="U$3" library="microbuilder" package="MOUNTINGHOLE_2.5_PLATED" value="MOUNTINGHOLE2.5" x="42.653" y="1.348" smashed="yes"/>
 <element name="U$4" library="microbuilder" package="MOUNTINGHOLE_2.5_PLATED" value="MOUNTINGHOLE2.5" x="42.888" y="29.1315" smashed="yes"/>
-<element name="U$5" library="oledBoard" package="SM04B-GHS-TB" value="SM04B-GHS-TB" x="45.339" y="23.7363" smashed="yes" rot="R90"/>
 <element name="U$6" library="oledBoard" package="CSTNE16M0VH3C000R0" value="CSTNE16M0VH3C000R0" x="24.436" y="9.8038" smashed="yes" rot="R90"/>
 <element name="U$8" library="oledBoard" package="SM03B-GHS-TB" value="SM03B-GHS-TB" x="45.212" y="7.6073" smashed="yes" rot="R90"/>
@@
 <attribute name="MF" value="" x="30.48" y="4.064" size="1.778" layer="27" rot="R180" display="off"/>
 <attribute name="MPN" value="" x="30.48" y="4.064" size="1.778" layer="27" rot="R180" display="off"/>
-<attribute name="NAME" x="34.29" y="1.143" size="1.27" layer="25" ratio="10" rot="R180"/>
 <attribute name="OC_FARNELL" value="unknown" x="30.48" y="4.064" size="1.778" layer="27" rot="R180" display="off"/>
 <attribute name="OC_NEWARK" value="unknown" x="30.48" y="4.064" size="1.778" layer="27" rot="R180" display="off"/>
@@
 <attribute name="VALUE" x="31.75" y="8.255" size="1.27" layer="27" ratio="10" rot="R180"/>
 </element>
+<element name="U$5" library="oledBoard" package="SM03B-GHS-TB" value="SM03B-GHS-TB" x="45.1612" y="16.2941" smashed="yes" rot="R90"/>
 </elements>
 <signals>
@@
 <via x="17.018" y="18.796" extent="1-16" drill="0.45"/>
 <contactref element="U$8" pad="P$5"/>
-<contactref element="U$5" pad="1"/>
 <wire x1="22.2535" y1="26.0033" x2="22.2535" y2="26.8255" width="0.254" layer="1"/>
 <contactref element="U5" pad="2"/>
@@
 <wire x1="-1.8772" y1="12.954" x2="-1.016" y2="12.954" width="0.3048" layer="1"/>
 <contactref element="SV1" pad="6"/>
+<contactref element="U$5" pad="P$5"/>
 <wire x1="28.7305" y1="26.0263" x2="28.2765" y2="26.0263" width="0" layer="19" extent="1-1"/>
 <wire x1="29.2305" y1="26.0263" x2="28.7765" y2="26.0263" width="0" layer="19" extent="1-1"/>
@@
 </signal>
 <signal name="AMMO1">
-<contactref element="U$5" pad="4"/>
 <contactref element="U3" pad="25"/>
-<wire x1="40.589" y1="21.3863" x2="39.893" y2="20.6903" width="0.2032" layer="1"/>
-<wire x1="35.7508" y1="17.9539" x2="33.2685" y2="17.9539" width="0.2032" layer="1"/>
-<wire x1="39.893" y1="20.6903" x2="38.4872" y2="20.6903" width="0.2032" layer="1"/>
-<wire x1="38.4872" y1="20.6903" x2="35.7508" y2="17.9539" width="0.2032" layer="1"/>
+<contactref element="U$5" pad="P$4"/>
+<wire x1="40.6112" y1="19.8941" x2="35.2087" y2="19.8941" width="0.2032" layer="1"/>
+<wire x1="35.2087" y1="19.8941" x2="33.2685" y2="17.9539" width="0.2032" layer="1"/>
 </signal>
 <signal name="AMMO2">
 <contactref element="U3" pad="24"/>
-<contactref element="U$5" pad="3"/>
-<wire x1="34.7611" y1="16.4613" x2="38.4361" y2="20.1363" width="0.2032" layer="1"/>
-<wire x1="38.4361" y1="20.1363" x2="40.589" y2="20.1363" width="0.2032" layer="1"/>
+<contactref element="U$5" pad="P$3"/>
+<wire x1="40.6112" y1="18.6441" x2="38.4284" y2="16.4613" width="0.2032" layer="1"/>
+<wire x1="38.4284" y1="16.4613" x2="34.7611" y2="16.4613" width="0.2032" layer="1"/>
 </signal>
 <signal name="AMMO3">
-<contactref element="U$5" pad="2"/>
 <contactref element="U3" pad="23"/>
-<wire x1="40.589" y1="18.8863" x2="40.1177" y2="18.415" width="0.2032" layer="1"/>
-<wire x1="36.2353" y1="15.6613" x2="34.7611" y2="15.6613" width="0.2032" layer="1"/>
-<wire x1="40.1177" y1="18.415" x2="38.989" y2="18.415" width="0.2032" layer="1"/>
-<wire x1="38.989" y1="18.415" x2="36.2353" y2="15.6613" width="0.2032" layer="1"/>
 </signal>
 <signal name="D-">
