File: Heads-Up-Display-ToF/Atmega328pTest/atmega328pTest.brd (EAGLE design)
At the start: 160 x 100 mm, 24 parts, among them IC1 FT232RL, P1 0475890001, U1 ATMEGA328P_TQFP

Commit message: update
Parts:
- moved C5 15.0 mm to (12.6, 19.5), turned to 180 degrees
- moved R5 3.66 mm to (28.8, 17.5), turned to 180 degrees
- moved R6 3.18 mm to (28.6, 14.6), turned to 180 degrees
Routing:
- net N$7: track 0.00 -> 3.80 mm
Changed lines of the file:
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@@
 <?xml version="1.0" encoding="utf-8"?>
 <!DOCTYPE eagle SYSTEM "eagle.dtd">
-<eagle version="9.5.2">
+<eagle version="9.5.0">
 <drawing>
 <settings>
@@
 <attribute name="VALUE" x="46.99" y="60.96" size="1.27" layer="27" rot="R180"/>
 </element>
-<element name="C5" library="rcl" library_urn="urn:adsk.eagle:library:334" package="C0603" package3d_urn="urn:adsk.eagle:package:23616/2" value="100nF" x="27.305" y="22.86" smashed="yes">
-<attribute name="NAME" x="26.67" y="23.495" size="1.27" layer="25"/>
-<attribute name="POPULARITY" value="37" x="45.085" y="-8.89" size="1.778" layer="27" display="off"/>
-<attribute name="SPICEPREFIX" value="C" x="45.085" y="-8.89" size="1.778" layer="27" display="off"/>
-<attribute name="VALUE" x="26.67" y="20.955" size="1.27" layer="27"/>
+<element name="C5" library="rcl" library_urn="urn:adsk.eagle:library:334" package="C0603" package3d_urn="urn:adsk.eagle:package:23616/2" value="100nF" x="12.6492" y="19.4564" smashed="yes" rot="R180">
+<attribute name="NAME" x="13.2842" y="18.8214" size="1.27" layer="25" rot="R180"/>
+<attribute name="POPULARITY" value="37" x="-5.1308" y="51.2064" size="1.778" layer="27" rot="R180" display="off"/>
+<attribute name="SPICEPREFIX" value="C" x="-5.1308" y="51.2064" size="1.778" layer="27" rot="R180" display="off"/>
+<attribute name="VALUE" x="13.2842" y="21.3614" size="1.27" layer="27" rot="R180"/>
 </element>
 <element name="C7" library="rcl" library_urn="urn:adsk.eagle:library:334" package="C0603" package3d_urn="urn:adsk.eagle:package:23616/2" value="100nF" x="97.79" y="20.32" smashed="yes" rot="R90">
@@
 <attribute name="VALUE" x="48.26" y="64.135" size="1.27" layer="27" rot="R270"/>
 </element>
-<element name="R5" library="rcl" library_urn="urn:adsk.eagle:library:334" package="R0603" package3d_urn="urn:adsk.eagle:package:23555/3" value="1K" x="31.75" y="19.685" smashed="yes">
-<attribute name="NAME" x="31.115" y="20.32" size="1.27" layer="25"/>
-<attribute name="POPULARITY" value="77" x="54.61" y="-17.145" size="1.778" layer="27" display="off"/>
-<attribute name="SPICEPREFIX" value="R" x="54.61" y="-17.145" size="1.778" layer="27" display="off"/>
-<attribute name="VALUE" x="31.115" y="17.78" size="1.27" layer="27"/>
-</element>
-<element name="R6" library="rcl" library_urn="urn:adsk.eagle:library:334" package="R0603" package3d_urn="urn:adsk.eagle:package:23555/3" value="1K" x="31.75" y="14.605" smashed="yes">
-<attribute name="NAME" x="31.115" y="15.24" size="1.27" layer="25"/>
-<attribute name="POPULARITY" value="77" x="58.42" y="-22.225" size="1.778" layer="27" display="off"/>
-<attribute name="SPICEPREFIX" value="R" x="58.42" y="-22.225" size="1.778" layer="27" display="off"/>
-<attribute name="VALUE" x="31.115" y="12.7" size="1.27" layer="27"/>
+<element name="R5" library="rcl" library_urn="urn:adsk.eagle:library:334" package="R0603" package3d_urn="urn:adsk.eagle:package:23555/3" value="1K" x="28.829" y="17.4752" smashed="yes" rot="R180">
+<attribute name="NAME" x="29.464" y="16.8402" size="1.27" layer="25" rot="R180"/>
+<attribute name="POPULARITY" value="77" x="5.969" y="54.3052" size="1.778" layer="27" rot="R180" display="off"/>
+<attribute name="SPICEPREFIX" value="R" x="5.969" y="54.3052" size="1.778" layer="27" rot="R180" display="off"/>
+<attribute name="VALUE" x="29.464" y="19.3802" size="1.27" layer="27" rot="R180"/>
+</element>
+<element name="R6" library="rcl" library_urn="urn:adsk.eagle:library:334" package="R0603" package3d_urn="urn:adsk.eagle:package:23555/3" value="1K" x="28.575" y="14.605" smashed="yes" rot="R180">
+<attribute name="NAME" x="29.21" y="13.97" size="1.27" layer="25" rot="R180"/>
+<attribute name="POPULARITY" value="77" x="1.905" y="51.435" size="1.778" layer="27" rot="R180" display="off"/>
+<attribute name="SPICEPREFIX" value="R" x="1.905" y="51.435" size="1.778" layer="27" rot="R180" display="off"/>
+<attribute name="VALUE" x="29.21" y="16.51" size="1.27" layer="27" rot="R180"/>
 </element>
 <element name="SV1" library="con-lstb" library_urn="urn:adsk.eagle:library:162" package="MA03-2" package3d_urn="urn:adsk.eagle:package:8334/1" value="ISO" x="120.65" y="40.005" smashed="yes">
@@
 <wire x1="56.5244" y1="51.015" x2="56.522" y2="51.0174" width="0.3048" layer="1"/>
 <wire x1="61.36" y1="55.3974" x2="123.19" y2="38.735" width="0" layer="19" extent="1-1"/>
-<wire x1="28.155" y1="22.86" x2="56.522" y2="51.0174" width="0" layer="19" extent="1-1"/>
+<wire x1="11.7992" y1="19.4564" x2="56.522" y2="51.0174" width="0" layer="19" extent="1-1"/>
 </signal>
 <signal name="N$1">
@@
 <contactref element="IC1" pad="2"/>
 <contactref element="C5" pad="1"/>
-<wire x1="17.299" y1="19.45" x2="26.455" y2="22.86" width="0" layer="19" extent="1-1"/>
+<wire x1="13.4992" y1="19.4564" x2="17.2926" y2="19.4564" width="0.254" layer="1"/>
+<wire x1="17.2926" y1="19.4564" x2="17.299" y2="19.45" width="0.254" layer="1"/>
 </signal>
 <signal name="N$5">
 <contactref element="IC1" pad="23"/>
 <contactref element="R5" pad="2"/>
-<wire x1="24.611" y1="16.85" x2="32.6" y2="19.685" width="0" layer="19" extent="1-1"/>
+<wire x1="24.611" y1="16.85" x2="27.979" y2="17.4752" width="0" layer="19" extent="1-1"/>
 </signal>
 <signal name="N$6">
 <contactref element="IC1" pad="22"/>
 <contactref element="R6" pad="2"/>
-<wire x1="24.611" y1="16.2" x2="32.6" y2="14.605" width="0" layer="19" extent="1-1"/>
+<wire x1="27.725" y1="14.605" x2="24.611" y2="16.2" width="0" layer="19" extent="1-1"/>
 </signal>
 <signal name="N$10">
 <contactref element="R5" pad="1"/>
 <contactref element="D2" pad="C"/>
-<wire x1="30.9" y1="19.685" x2="38.977" y2="20.955" width="0" layer="19" extent="1-1"/>
+<wire x1="29.679" y1="17.4752" x2="38.977" y2="20.955" width="0" layer="19" extent="1-1"/>
 </signal>
 <signal name="N$11">
 <contactref element="R6" pad="1"/>
 <contactref element="D3" pad="C"/>
-<wire x1="30.9" y1="14.605" x2="39.612" y2="14.605" width="0" layer="19" extent="1-1"/>
+<wire x1="29.425" y1="14.605" x2="39.612" y2="14.605" width="0" layer="19" extent="1-1"/>
 </signal>
 <signal name="N$8">

Commit message: OLED board update
Parts:
- removed C3, C8: 4.7uF 16V, rcl:C1206
- removed D4: Yellow, SparkFun-LED:LED-0603
- added C18, C19, C20, C21, C22, C23: 0.1uF, SparkFun-Capacitors:0603
- added D8: GREEN, SparkFun-LED:LED-0603
- added D9: 1A/23V/620mV, SparkFun-DiscreteSemi:SOD-323
- added L2: 4.7µH/±30%/1.2A, SparkFun-Coils:INDUCTOR_4.7UH
- added R21: 1k, SparkFun-Resistors:0603
- added R22: 47k, SparkFun-Resistors:0603
- added R23: 5.6k, SparkFun-Resistors:0603
- added R24: 100k, SparkFun-Resistors:0603
- added R7, R8: 10K, rcl:R0603
- added U$13, U$14: SM03B-GHS-TB, oledBoard:SM03B-GHS-TB
- added U$15: XT30PW-M, oledBoard:XT30
- added U7: AP3012, SparkFun-IC-Power:SOT23-5
- added U8: UG-2856KLBAG01_4WSPI, SparkFun-Displays:FPC05024-42201
- moved P1 89.8 mm to (56.6, 89.9), turned to 180 degrees
- moved C5 75.9 mm to (64.8, 74.5), turned to 0 degrees
- moved IC1 71.7 mm to (56.5, 78.1), turned to 90 degrees
- moved C7 70.2 mm to (64.1, 81.9), turned to 270 degrees
- moved R6 67.9 mm to (48.7, 79.4), turned to 0 degrees
- moved D3 65.0 mm to (43.8, 79.4)
- moved R5 62.3 mm to (48.6, 76.5), turned to 0 degrees
- moved U$3 61.7 mm to (68.6, 79.4), turned to 90 degrees
- moved SV1 61.7 mm to (59.1, 43.2), turned to 180 degrees
- moved D2 55.8 mm to (43.8, 76.5)
- moved C2 25.0 mm to (68.6, 53.3), turned to 0 degrees
- moved U$2 24.3 mm to (65.9, 67.8), turned to 180 degrees
- moved U$1 24.1 mm to (46.6, 54.7), turned to 90 degrees
- moved D1 23.0 mm to (64.8, 50.2), turned to 270 degrees
- moved C4 22.2 mm to (68.6, 59.1), turned to 0 degrees
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Connections:
- removed net 3V3OUT: IC1.17
- removed net N$12: D4.A, U1.10
- new net 12V: C19.1, C20.1, C21.1, D9.C, R22.2, U8.P$23
- new net 3.3V: C18.1, C22.1, IC1.17, L2.P$1, U7.4, U7.5
- new net AMMO1: U$14.P$4
- new net AMMO2: U$14.P$3
- new net N$27: D8.C, R21.2
- new net N$28: D9.A, L2.P$2, U7.1
- new net N$29: R22.1, R23.2, U7.3
- new net N$30: C23.1, U8.P$22
- new net N$31: R24.2, U8.P$21
- new net PC0: U1.23
- new net PC1: U1.24
- new net PC2: U1.25
- new net SCL: R8.2, U1.28, U8.P$13
- new net SDA: R7.2, U1.27, U8.P$14, U8.P$15
- new net VCC: U$15.P$1, U8.P$5, U8.P$6
- net +5V: now also D8.A, R7.1, R8.1; no longer C8.1
- net GND: now also C18.2, C19.2, C20.2, C21.2, C22.2, C23.2, R21.1, R23.1, R24.1, U$13.P$5, U$14.P$5, U$15.P$2, U7.2, U8.P$1, U8.P$10, U8.P$11, U8.P$12, U8.P$16, U8.P$17, U8.P$18, U8.P$19, U8.P$2, U8.P$20, U8.P$24, U8.P$3, U8.P$7, U8.P$8; no longer C3.2, C8.2, D4.C
- net RX: now also U$13.P$3
- net TX: now also U$13.P$4
- net VUSB: no longer C3.1
Routing:
- net RESET: track 7.87 -> 37.8 mm, vias 0 -> 2
- net SCL: track 0.00 -> 20.4 mm
- net +5V: track 25.2 -> 42.7 mm, vias 4 -> 7
- net 3.3V: track 0.00 -> 13.9 mm, vias 0 -> 1
- net PC0: track 0.00 -> 13.7 mm
- net MOSI: track 0.00 -> 13.5 mm
- net SDA: track 0.00 -> 13.0 mm
- net TX: track 0.00 -> 12.0 mm
- net PC1: track 0.00 -> 11.7 mm
- net MISO: track 0.00 -> 11.7 mm
- net PC2: track 0.00 -> 11.7 mm
- net SCK: track 6.57 -> 18.1 mm, vias 0 -> 2
- net RX: track 0.00 -> 9.47 mm
- net D-: track 0.00 -> 7.78 mm
- net D+: track 0.00 -> 6.48 mm
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- added copper zone on layer 1, net 12V
- added copper zone on layer 1, net 5V
- added copper zone on layer 1, net N$13
- added copper zone on layer 1, net N$14
- added copper zone on layer 1, net N$26
- added copper zone on layer 1, net VCC
- added copper zone on layer 16, net VCC
Other:
- board size 160 x 100 mm -> 94.1 x 131.1 mm
- board text added: "3.3V"
- board text added: "ATMEGA328P Test Board"
- board text added: "CS"
- board text added: "GND"
- board text added: "MISO"
- board text added: "MOSI"
- board text added: "PC0"
- board text added: "PC1"
- board text added: "PC2"
- board text added: "RX"
- board text added: "Robomaster OLED Control Board V1.1 By Henry Silva 11/6/2019"
- board text added: "SCL"
- board text added: "SDA"
- board text added: "VCC"
