File: Heads-Up-Display-ToF/Atmega328pTest/atmega328pTest.sch (EAGLE design)
At the start: 23 parts, among them IC1 FT232RL, P1 0475890001, U1 ATMEGA328P_TQFP

Commit message: test board update
Parts:
- removed C6: 4.7uF 16V, rcl:C-USC0603
- added C8: 4.7uF 16V, rcl:C-USC1206
- added D4: Yellow, SparkFun-LED:LED0603
- C3: device rcl:C-USC0603 -> rcl:C-USC1206
- SV1: value (none) -> ISO
Connections:
- new net N$12: D4.A, U1.PD6(AIN0)
- net +5V: now also C8.1; no longer C3.1
- net GND: now also C8.2, D4.C; no longer C6.2
- net VUSB: now also C3.1; no longer C6.1
Other:
- moved on the sheet: C3
Changed lines of the file:
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@@
 <part name="P+1" library="supply1" library_urn="urn:adsk.eagle:library:371" deviceset="+5V" device=""/>
 <part name="C2" library="rcl" library_urn="urn:adsk.eagle:library:334" deviceset="C-US" device="C0603" package3d_urn="urn:adsk.eagle:package:23616/2" value="1uF"/>
-<part name="C3" library="rcl" library_urn="urn:adsk.eagle:library:334" deviceset="C-US" device="C0603" package3d_urn="urn:adsk.eagle:package:23616/2" value="4.7uF 16V"/>
 <part name="C4" library="rcl" library_urn="urn:adsk.eagle:library:334" deviceset="C-US" device="C0603" package3d_urn="urn:adsk.eagle:package:23616/2" value="1uF"/>
 <part name="GND4" library="supply1" library_urn="urn:adsk.eagle:library:371" deviceset="GND" device=""/>
@@
 <part name="U$3" library="HenrySilva" deviceset="SS1P3L-M3/84A" device=""/>
 <part name="P+5" library="supply1" library_urn="urn:adsk.eagle:library:371" deviceset="+5V" device=""/>
-<part name="C6" library="rcl" library_urn="urn:adsk.eagle:library:334" deviceset="C-US" device="C0603" package3d_urn="urn:adsk.eagle:package:23616/2" value="4.7uF 16V"/>
 <part name="C7" library="rcl" library_urn="urn:adsk.eagle:library:334" deviceset="C-US" device="C0603" package3d_urn="urn:adsk.eagle:package:23616/2" value="100nF"/>
 <part name="GND9" library="supply1" library_urn="urn:adsk.eagle:library:371" deviceset="GND" device=""/>
-<part name="SV1" library="con-lstb" library_urn="urn:adsk.eagle:library:162" deviceset="MA03-2" device="" package3d_urn="urn:adsk.eagle:package:8334/1"/>
+<part name="SV1" library="con-lstb" library_urn="urn:adsk.eagle:library:162" deviceset="MA03-2" device="" package3d_urn="urn:adsk.eagle:package:8334/1" value="ISO"/>
 <part name="P+6" library="supply1" library_urn="urn:adsk.eagle:library:371" deviceset="+5V" device=""/>
 <part name="GND10" library="supply1" library_urn="urn:adsk.eagle:library:371" deviceset="GND" device=""/>
+<part name="D4" library="SparkFun-LED" deviceset="LED" device="0603" value="Yellow"/>
+<part name="GND11" library="supply1" library_urn="urn:adsk.eagle:library:371" deviceset="GND" device=""/>
+<part name="C8" library="rcl" library_urn="urn:adsk.eagle:library:334" deviceset="C-US" device="C1206" package3d_urn="urn:adsk.eagle:package:23618/2" value="4.7uF 16V"/>
+<part name="C3" library="rcl" library_urn="urn:adsk.eagle:library:334" deviceset="C-US" device="C1206" package3d_urn="urn:adsk.eagle:package:23618/2" value="4.7uF 16V"/>
 </parts>
 <sheets>
@@
 <attribute name="VALUE" x="-67.564" y="-32.131" size="1.778" layer="96"/>
 </instance>
-<instance part="C3" gate="G$1" x="-58.42" y="-27.94" smashed="yes">
-<attribute name="NAME" x="-57.404" y="-27.305" size="1.778" layer="95"/>
-<attribute name="VALUE" x="-57.404" y="-32.131" size="1.778" layer="96"/>
-</instance>
 <instance part="C4" gate="G$1" x="-45.72" y="-27.94" smashed="yes">
 <attribute name="NAME" x="-44.704" y="-27.305" size="1.778" layer="95"/>
@@
 <attribute name="VALUE" x="96.52" y="-91.44" size="1.778" layer="96" rot="R90"/>
 </instance>
-<instance part="C6" gate="G$1" x="177.8" y="-88.9" smashed="yes">
-<attribute name="NAME" x="178.816" y="-88.265" size="1.778" layer="95"/>
-<attribute name="VALUE" x="178.816" y="-93.091" size="1.778" layer="96"/>
-</instance>
 <instance part="C7" gate="G$1" x="193.04" y="-88.9" smashed="yes">
 <attribute name="NAME" x="194.056" y="-88.265" size="1.778" layer="95"/>
@@
 <instance part="GND10" gate="1" x="160.02" y="-71.12" smashed="yes">
 <attribute name="VALUE" x="157.48" y="-73.66" size="1.778" layer="96"/>
+</instance>
+<instance part="D4" gate="D1" x="68.58" y="-45.72" smashed="yes" rot="MR270">
+<attribute name="NAME" x="73.152" y="-42.291" size="1.778" layer="95" font="vector" rot="MR0"/>
+<attribute name="VALUE" x="73.152" y="-47.625" size="1.778" layer="96" font="vector" rot="MR0" align="top-left"/>
+</instance>
+<instance part="GND11" gate="1" x="81.28" y="-50.8" smashed="yes">
+<attribute name="VALUE" x="78.74" y="-53.34" size="1.778" layer="96"/>
+</instance>
+<instance part="C8" gate="G$1" x="-58.42" y="-27.94" smashed="yes">
+<attribute name="NAME" x="-57.404" y="-27.305" size="1.778" layer="95"/>
+<attribute name="VALUE" x="-57.404" y="-32.131" size="1.778" layer="96"/>
+</instance>
+<instance part="C3" gate="G$1" x="177.8" y="-88.9" smashed="yes">
+<attribute name="NAME" x="178.816" y="-88.265" size="1.778" layer="95"/>
+<attribute name="VALUE" x="178.816" y="-93.091" size="1.778" layer="96"/>
 </instance>
 </instances>
@@
 <pinref part="C4" gate="G$1" pin="2"/>
 <wire x1="-45.72" y1="-33.02" x2="-45.72" y2="-35.56" width="0.1524" layer="91"/>
-<pinref part="C3" gate="G$1" pin="2"/>
 <wire x1="-45.72" y1="-35.56" x2="-45.72" y2="-38.1" width="0.1524" layer="91"/>
 <wire x1="-58.42" y1="-33.02" x2="-58.42" y2="-35.56" width="0.1524" layer="91"/>
@@
 <junction x="-58.42" y="-35.56"/>
 <pinref part="GND4" gate="1" pin="GND"/>
+<pinref part="C8" gate="G$1" pin="2"/>
 </segment>
 <segment>
@@
 </segment>
 <segment>
-<pinref part="C6" gate="G$1" pin="2"/>
 <wire x1="177.8" y1="-93.98" x2="177.8" y2="-99.06" width="0.1524" layer="91"/>
 <wire x1="177.8" y1="-99.06" x2="185.42" y2="-99.06" width="0.1524" layer="91"/>
@@
 <junction x="185.42" y="-99.06"/>
 <pinref part="GND9" gate="1" pin="GND"/>
+<pinref part="C3" gate="G$1" pin="2"/>
 </segment>
 <segment>
@@
 <wire x1="160.02" y1="-66.04" x2="160.02" y2="-68.58" width="0.1524" layer="91"/>
 <pinref part="GND10" gate="1" pin="GND"/>
+</segment>
+<segment>
+<pinref part="D4" gate="D1" pin="C"/>
+<wire x1="73.66" y1="-45.72" x2="81.28" y2="-45.72" width="0.1524" layer="91"/>
+<wire x1="81.28" y1="-45.72" x2="81.28" y2="-48.26" width="0.1524" layer="91"/>
+<pinref part="GND11" gate="1" pin="GND"/>
 </segment>
 </net>
@@
 <pinref part="C4" gate="G$1" pin="1"/>
 <wire x1="-45.72" y1="-20.32" x2="-45.72" y2="-25.4" width="0.1524" layer="91"/>
-<pinref part="C3" gate="G$1" pin="1"/>
 <wire x1="-58.42" y1="-20.32" x2="-58.42" y2="-25.4" width="0.1524" layer="91"/>
 <pinref part="C2" gate="G$1" pin="1"/>
 <wire x1="-68.58" y1="-20.32" x2="-68.58" y2="-25.4" width="0.1524" layer="91"/>
+<pinref part="C8" gate="G$1" pin="1"/>
 </segment>
 <segment>
@@
 </segment>
 <segment>
-<pinref part="C6" gate="G$1" pin="1"/>
 <wire x1="177.8" y1="-86.36" x2="177.8" y2="-81.28" width="0.1524" layer="91"/>
 <wire x1="177.8" y1="-81.28" x2="185.42" y2="-81.28" width="0.1524" layer="91"/>
@@
 <junction x="185.42" y="-81.28"/>
 <label x="185.42" y="-76.2" size="1.778" layer="95"/>
-</segment>
-</net>
+<pinref part="C3" gate="G$1" pin="1"/>
+</segment>
+</net>
+<net name="N$12" class="0">
+<segment>
+<pinref part="U1" gate="U1" pin="PD6(AIN0)"/>
+<wire x1="58.42" y1="-45.72" x2="66.04" y2="-45.72" width="0.1524" layer="91"/>
+<pinref part="D4" gate="D1" pin="A"/>
+</segment>
+</net>

Commit message: OLED board update
Parts:
- removed C3, C8: 4.7uF 16V, rcl:C-USC1206
- removed D4: Yellow, SparkFun-LED:LED0603
- added C18, C19, C20, C21, C22, C23: 0.1uF, SparkFun-Capacitors:0.1UF-0603-25V-(+80/-20%)
- added D8: GREEN, SparkFun-LED:LED0603
- added D9: 1A/23V/620mV, SparkFun-DiscreteSemi:DIODE-SCHOTTKY-BAT20J
- added L2: 4.7µH/±30%/1.2A, SparkFun-Coils:INDUCTOR-CDRH-4.7UH
- added R21: 1k, SparkFun-Resistors:1KOHM-0603-1/10W-1%
- added R22: 47k, SparkFun-Resistors:47KOHM-0603-1/10W-1%
- added R23: 5.6k, SparkFun-Resistors:5.6KOHM-0603-1/10W-1%
- added R24: 100k, SparkFun-Resistors:100KOHM-0603-1/10W-1%
- added R7, R8: 10K, rcl:R-US_R0603
- added U$13, U$14: SM03B-GHS-TB, oledBoard:SM03B-GHS-TB
- added U$15: XT30PW-M, oledBoard:XT30PW-M
- added U7: AP3012, SparkFun-IC-Power:AP3012
- added U8: UG-2856KLBAG01_4WSPI, SparkFun-Displays:UG-2856KLBAG01_4WSPI
Connections:
- removed net N$12: D4.A, U1.PD6(AIN0)
- new net 12V: C19.1, C20.1, C21.1, D9.C, R22.2, U8.VCC
- new net 3.3V: C18.1, C22.1, IC1.3V3OUT, L2.1, U7.!SHDN!, U7.VIN
- new net AMMO1: U$14.2
- new net AMMO2: U$14.1
- new net N$27: D8.C, R21.2
- new net N$28: D9.A, L2.2, U7.SW
- new net N$29: R22.1, R23.2, U7.FB
- new net N$30: C23.1, U8.VCOMH
- new net N$31: R24.2, U8.IREF
- new net PC0: U1.PC0(ADC0)
- new net PC1: U1.PC1(ADC1)
- new net PC2: U1.PC2(ADC2)
- new net SCL: R8.2, U1.PC5(ADC5/SCL), U8.SCLK/SCL
- new net SDA: R7.2, U1.PC4(ADC4/SDA), U8.NC/D2, U8.SDIN/SDA
- new net VCC: U$15.VCC, U8.BS1, U8.VDD
- net +5V: now also D8.A, R7.1, R8.1; no longer C8.1
- net GND: now also C18.2, C19.2, C20.2, C21.2, C22.2, C23.2, R21.1, R23.1, R24.1, U$13.3, U$14.3, U$15.GND, U7.GND, U8.!CS, U8.BS2, U8.D!C!/SA0, U8.GND, U8.VLSS, U8.VSS; no longer C3.2, C8.2, D4.C
- net RX: now also U$13.1
- net TX: now also U$13.2
- net VUSB: no longer C3.1
Other:
- note added: "Atmega"
- note added: "Boost 3.3v -> 12v"
- note added: "Connectors"
- note added: "ISP"
- note added: "OLED"
- note added: "USB"
- note added: "USB To Serial"
- moved on the sheet: C1, C2, C4, C5, C7, D1, D2, D3, IC1, P1, R1, R2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
