File: Low-Ammo Detector/RingBoardV2/hopperBoardV2.brd (EAGLE design)
At the start: 172.2 x 172.3 mm, 17 parts

Commit message: Ammo Board V2
Parts:
- removed U$10, U$11, U$12, U$7: MOUNTINGHOLE3.0THIN, microbuilder:MOUNTINGHOLE_3.0_PLATEDTHIN
- R1: value 540k -> 330k
- R2: value 360k -> 180k
- U$6: value XT30PW-M -> SM02B-GHS-TB; device _HenrySilva:XT30 -> _HenrySilva:SM02B-GHS-TB
- moved U$2 18.0 mm to (-1.23, 65.1)
- moved U$1 17.1 mm to (64.0, 1.28), turned to 270 degrees
- moved U$3 15.0 mm to (2.00, -68.0)
- moved U$4 15.0 mm to (-68.0, -2.00)
- moved U$8 12.4 mm to (65.0, -30.0)
- moved C1 10.8 mm to (64.0, -13.2)
- moved C2 10.8 mm to (66.5, -7.19)
- moved C3 10.8 mm to (66.5, -3.69)
- moved R1 10.8 mm to (69.0, -7.19)
- moved R2 10.8 mm to (69.0, -10.7)
- moved U$5 10.8 mm to (63.0, -11.2)
- moved U$9 10.8 mm to (63.0, -6.19)
- moved U$6 7.83 mm to (67.0, -22.0), turned to 90 degrees
Connections:
- net 5V: now also U$6.P$3; no longer U$6.P$1
- net GND: now also U$6.P$4; no longer U$6.P$2
Routing:
- net AMMO1: track 159.7 -> 131.8 mm
- net AMMO2: track 93.1 -> 73.3 mm
- net 1.5V: track 116.9 -> 101.4 mm
- net 5V: track 1.26 -> 3.77 mm, vias 7 -> 8
Other:
- board size 172.2 x 172.3 mm -> 144 x 146.5 mm
- board text added: "Purdue Robomaster Ammo Sensor Board V2.0 By Henry Silva 12/7/2019"
- board text removed: "Purdue Robomaster Ammo Sensor Board V1.0 By Henry Silva 11/9/2019"

Commit message: OLED board update
Parts:
- moved U$3 3.61 mm to (0.00, -65.0), turned to 135 degrees
- moved U$4 3.61 mm to (-65.0, 0.00), turned to 135 degrees
- moved U$1 1.60 mm to (65.0, 0.01), turned to 315 degrees
- moved U$2 1.22 mm to (-0.01, 65.0), turned to 315 degrees
Connections:
- net AMMO1: now also U$3.P$2; no longer U$4.P$2
- net AMMO2: now also U$4.P$2; no longer U$3.P$2
Routing:
- net AMMO2: track 73.3 -> 134.9 mm
- net AMMO1: track 131.8 -> 73.8 mm
- net 1.5V: track 101.4 -> 98.1 mm
Changed lines of the file:
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@@
 <setting verticaltext="up"/>
 </settings>
-<grid distance="39.3700787" unitdist="mil" unit="mil" style="lines" multiple="1" display="yes" altdistance="5" altunitdist="mil" altunit="mil"/>
+<grid distance="1" unitdist="mm" unit="mm" style="lines" multiple="1" display="yes" altdistance="1" altunitdist="mil" altunit="mil"/>
 <layers>
 <layer number="1" name="Top" color="4" fill="1" visible="yes" active="yes"/>
@@
 </autorouter>
 <elements>
-<element name="U$3" library="_HenrySilva" package="OPL550" value="OPL550" x="2" y="-68" smashed="yes" rot="R180"/>
-<element name="U$4" library="_HenrySilva" package="OPL550" value="OPL550" x="-68" y="-2" smashed="yes" rot="R90"/>
+<element name="U$3" library="_HenrySilva" package="OPL550" value="OPL550" x="0" y="-65" smashed="yes" rot="R135"/>
+<element name="U$4" library="_HenrySilva" package="OPL550" value="OPL550" x="-65" y="0" smashed="yes" rot="R135"/>
 <element name="U$5" library="_HenrySilva" package="TPS62260" value="TPS62260" x="62.964" y="-11.1904" smashed="yes"/>
-<element name="U$1" library="_HenrySilva" package="2PIN" value="2PIN" x="64.0368" y="1.2768" smashed="yes" rot="R270"/>
-<element name="U$2" library="_HenrySilva" package="2PIN" value="2PIN" x="-1.226" y="65.102" smashed="yes"/>
+<element name="U$1" library="_HenrySilva" package="2PIN" value="2PIN" x="65.0114" y="0.0068" smashed="yes" rot="R315"/>
+<element name="U$2" library="_HenrySilva" package="2PIN" value="2PIN" x="-0.0068" y="65.0004" smashed="yes" rot="R315"/>
 <element name="U$8" library="_HenrySilva" package="SM03B-GHS-TB" value="SM03B-GHS-TB" x="65" y="-30" smashed="yes" rot="R90"/>
 <element name="C1" library="rcl" library_urn="urn:adsk.eagle:library:334" package="C0603" package3d_urn="urn:adsk.eagle:package:23616/2" value="4.7uF" x="63.964" y="-13.1904" smashed="yes">
@@
 </signal>
 <signal name="AMMO2">
+<contactref element="U$8" pad="P$3"/>
+<wire x1="60.45" y1="-27.65" x2="60.45" y2="-30.99" width="0.2032" layer="1"/>
+<wire x1="60.45" y1="-30.99" x2="59.69" y2="-31.75" width="0.2032" layer="1"/>
+<contactref element="U$4" pad="P$2"/>
+<wire x1="59.69" y1="-31.75" x2="-65.024" y2="-2.286" width="0.2032" layer="1" curve="-154.533764"/>
+<wire x1="-65.024" y1="-2.286" x2="-65.024" y2="-0.033334375" width="0.2032" layer="1"/>
+<wire x1="-65.024" y1="-0.033334375" x2="-64.99533125" y2="-0.004665625" width="0.2032" layer="1"/>
+</signal>
+<signal name="AMMO1">
+<contactref element="U$8" pad="P$4"/>
+<wire x1="60.45" y1="-26.4" x2="60.434" y2="-26.416" width="0.2032" layer="1"/>
+<wire x1="60.434" y1="-26.416" x2="59.182" y2="-26.416" width="0.2032" layer="1"/>
+<wire x1="59.182" y1="-26.416" x2="58.42" y2="-27.178" width="0.2032" layer="1"/>
+<wire x1="58.42" y1="-27.178" x2="58.42" y2="-30.734" width="0.2032" layer="1"/>
 <contactref element="U$3" pad="P$2"/>
-<contactref element="U$8" pad="P$3"/>
-<wire x1="60.45" y1="-27.65" x2="59.35" y2="-27.65" width="0.2032" layer="1"/>
-<wire x1="59.35" y1="-27.65" x2="59" y2="-28" width="0.2032" layer="1"/>
-<wire x1="1" y1="-66" x2="59" y2="-28" width="0.2032" layer="1" curve="63.627489"/>
-<wire x1="0" y1="-68" x2="0" y2="-67" width="0.2032" layer="1"/>
-<wire x1="0" y1="-67" x2="1" y2="-66" width="0.2032" layer="1"/>
-</signal>
-<signal name="AMMO1">
-<contactref element="U$4" pad="P$2"/>
-<contactref element="U$8" pad="P$4"/>
-<wire x1="60.45" y1="-26.4" x2="58.6" y2="-26.4" width="0.2032" layer="1"/>
-<wire x1="58.6" y1="-26.4" x2="58" y2="-27" width="0.2032" layer="1"/>
-<wire x1="-65" y1="-1" x2="58" y2="-27" width="0.2032" layer="1" curve="152.646665"/>
-<wire x1="-68" y1="0" x2="-66" y2="0" width="0.2032" layer="1"/>
-<wire x1="-66" y1="0" x2="-65" y2="-1" width="0.2032" layer="1"/>
+<wire x1="58.42" y1="-30.734" x2="1.778" y2="-64.262" width="0.2032" layer="1" curve="-59.606986"/>
+<wire x1="1.778" y1="-64.262" x2="0.74733125" y2="-64.262" width="0.2032" layer="1"/>
+<wire x1="0.74733125" y1="-64.262" x2="0.004665625" y2="-65.004665625" width="0.2032" layer="1"/>
 </signal>
 <signal name="N$1">
@@
 <vertex x="64.406" y="-4.222"/>
 </polygon>
-<wire x1="64.0368" y1="-1.2232" x2="67.2232" y2="-1.2232" width="0.254" layer="1"/>
-<wire x1="67.2232" y1="-1.2232" x2="68" y2="-2" width="0.254" layer="1"/>
-<wire x1="68" y1="-2" x2="68" y2="-4" width="0.254" layer="1"/>
-<wire x1="3" y1="65" x2="68" y2="-2" width="0.254" layer="1" curve="-88.290186"/>
-<wire x1="1.274" y1="65.102" x2="2.898" y2="65.102" width="0.254" layer="1"/>
-<wire x1="2.898" y1="65.102" x2="3" y2="65" width="0.254" layer="1"/>
+<wire x1="68" y1="-2" x2="68" y2="-4" width="0.3048" layer="1"/>
+<wire x1="3" y1="65" x2="68" y2="-2" width="0.3048" layer="1" curve="-88.290186"/>
+<wire x1="3" y1="65" x2="1.2236" y2="65" width="0.3048" layer="1"/>
+<wire x1="0.862940625" y1="64.13065625" x2="1.2236" y2="65" width="0.3048" layer="1"/>
+<wire x1="66.464" y1="-4.5404" x2="65.881140625" y2="-0.862940625" width="0" layer="19" extent="1-1"/>
 </signal>
 </signals>
