File: Low-Ammo Detector/RingBoardV2/hopperBoardV2.sch (EAGLE design)
At the start: 16 parts

Commit message: Ammo Board V2
Parts:
- removed U$10, U$11, U$12, U$7: MOUNTINGHOLE3.0THIN, microbuilder:MOUNTINGHOLE3.0THIN
- added U$6: SM02B-GHS-TB, _HenrySilva:SM02B-GHS-TB
- R1: value 540k -> 330k
- R2: value 360k -> 180k
Connections:
- net 5V: now also U$6.1
- net GND: now also U$6.2
Changed lines of the file:
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@@
 <setting verticaltext="up"/>
 </settings>
-<grid distance="0.1" unitdist="inch" unit="inch" style="lines" multiple="1" display="yes" altdistance="0.01" altunitdist="inch" altunit="inch"/>
+<grid distance="0.1" unitdist="inch" unit="inch" style="lines" multiple="1" display="no" altdistance="0.01" altunitdist="inch" altunit="inch"/>
 <layers>
 <layer number="1" name="Top" color="4" fill="1" visible="no" active="no"/>
@@
 <part name="C2" library="rcl" library_urn="urn:adsk.eagle:library:334" deviceset="C-US" device="C0603" package3d_urn="urn:adsk.eagle:package:23616/2" value="22pF"/>
 <part name="C3" library="rcl" library_urn="urn:adsk.eagle:library:334" deviceset="C-US" device="C0603" package3d_urn="urn:adsk.eagle:package:23616/2" value="10uF"/>
-<part name="R1" library="rcl" library_urn="urn:adsk.eagle:library:334" deviceset="R-US_" device="R0603" package3d_urn="urn:adsk.eagle:package:23555/3" value="540k"/>
-<part name="R2" library="rcl" library_urn="urn:adsk.eagle:library:334" deviceset="R-US_" device="R0603" package3d_urn="urn:adsk.eagle:package:23555/3" value="360k"/>
-<part name="U$10" library="microbuilder" deviceset="MOUNTINGHOLE" device="3.0THIN"/>
-<part name="U$11" library="microbuilder" deviceset="MOUNTINGHOLE" device="3.0THIN"/>
-<part name="U$12" library="microbuilder" deviceset="MOUNTINGHOLE" device="3.0THIN"/>
-<part name="U$7" library="microbuilder" deviceset="MOUNTINGHOLE" device="3.0THIN"/>
+<part name="R1" library="rcl" library_urn="urn:adsk.eagle:library:334" deviceset="R-US_" device="R0603" package3d_urn="urn:adsk.eagle:package:23555/3" value="330k"/>
+<part name="R2" library="rcl" library_urn="urn:adsk.eagle:library:334" deviceset="R-US_" device="R0603" package3d_urn="urn:adsk.eagle:package:23555/3" value="180k"/>
+<part name="U$6" library="_HenrySilva" deviceset="SM02B-GHS-TB" device=""/>
 </parts>
 <sheets>
@@
 <attribute name="VALUE" x="165.862" y="-1.27" size="1.778" layer="96" rot="R90"/>
 </instance>
-<instance part="U$10" gate="G$1" x="43.18" y="2.54" smashed="yes"/>
-<instance part="U$11" gate="G$1" x="25.4" y="20.32" smashed="yes"/>
-<instance part="U$12" gate="G$1" x="43.18" y="20.32" smashed="yes"/>
-<instance part="U$7" gate="G$1" x="25.4" y="2.54" smashed="yes"/>
+<instance part="U$6" gate="G$1" x="-38.1" y="55.88" smashed="yes" rot="R90"/>
 </instances>
 <busses>
@@
 <wire x1="162.56" y1="-2.54" x2="162.56" y2="-5.08" width="0.1524" layer="91"/>
 <label x="162.56" y="-5.08" size="1.778" layer="95" rot="R270"/>
+</segment>
+<segment>
+<pinref part="U$6" gate="G$1" pin="2"/>
+<wire x1="-43.18" y1="50.8" x2="-43.18" y2="45.72" width="0.1524" layer="91"/>
+<label x="-43.18" y="45.72" size="1.778" layer="95" rot="R270"/>
 </segment>
 </net>
@@
 <label x="104.14" y="25.4" size="1.778" layer="95" rot="R180"/>
 </segment>
+<segment>
+<pinref part="U$6" gate="G$1" pin="1"/>
+<wire x1="-40.64" y1="50.8" x2="-40.64" y2="45.72" width="0.1524" layer="91"/>
+<label x="-40.64" y="45.72" size="1.778" layer="95" rot="R270"/>
+</segment>
 </net>

Commit message: OLED board update
Connections:
- net AMMO1: now also U$3.OUT; no longer U$4.OUT
- net AMMO2: now also U$4.OUT; no longer U$3.OUT
Other:
- note added: "IR Laser"
- moved on the sheet: C1, C2, C3, R1, R2, U$9
