File: Robomaster-Controller-Board-v4.0/Kevin's Version/RMCB4.brd (EAGLE design)
At the start: 57.5 x 49.2 mm, 98 parts, among them Q1 3.1A/30V/105mΩ, SW1 EG1319, U2 AP2112-3.3, X4 32.768, Y2 12mhz

Commit message: Updated Schematic
Parts:
- removed AUX_GPIO2: S2B-PH-SM4_TB, KevinMade:S2B-PH-SM4_TB
- removed I2C_3, I2C_6: SM04B-GHS-TB(LF)(SN)-, SM04B-GHS-TB_LF__SN_-:JST_SM04B-GHS-TB(LF)(SN)-
- added GPIO_AUX1, GPIO_AUX2: S2B-PH-SM4_TB, KevinMade:S2B-PH-SM4_TB
- renumbered PC1 to PC13
Connections:
- net D10 renamed PB9
- net D9 renamed PB8
- net MISO renamed PB14
- net MOSI renamed PB15
- net SCK renamed PB13
- removed net BACKUP2: AUX_GPIO2.1, STM32F405RGTX.25
- removed net D8_NEOPIX: NEO.1, STM32F405RGTX.8
- removed net I2C-3_CL: I2C_3.2, I2C_6.2, RN1.3, STM32F405RGTX.41
- removed net I2C-3_DA: I2C_3.3, I2C_6.3, RN1.4, STM32F405RGTX.40
- new net GPIO_AUX1: GPIO_AUX1.1, STM32F405RGTX.25
- new net GPIO_AUX2: GPIO_AUX2.1, STM32F405RGTX.24
- new net NEOPIX: NEO.1, STM32F405RGTX.41
- new net PC13: R12.1, STM32F405RGTX.2
- new net PC6: STM32F405RGTX.37
- new net PC7: STM32F405RGTX.38
- net 3.3V: no longer I2C_3.1, I2C_6.1, RN1.5, RN1.6, STM32F405RGTX.42, STM32F405RGTX.43
- net D13: no longer R12.1
- net D14: now also STM32F405RGTX.8; no longer STM32F405RGTX.24
- net GND: now also GPIO_AUX1.2, GPIO_AUX2.2; no longer AUX_GPIO2.2, I2C_3.4, I2C_6.4
- net SDIO_CLK: now also STM32F405RGTX.53; no longer STM32F405RGTX.38
- net SDIO_CMD: now also STM32F405RGTX.54; no longer STM32F405RGTX.37
- net SDIO_D1: now also STM32F405RGTX.40; no longer STM32F405RGTX.2
- net SHIELD: no longer I2C_3.SH1, I2C_3.SH2, I2C_6.SH1, I2C_6.SH2
- net VISION_RX: now also STM32F405RGTX.43; no longer STM32F405RGTX.54
- net VISION_TX: now also STM32F405RGTX.42; no longer STM32F405RGTX.53
Routing:
- net I2C-3_CL: track 65.1 -> 0.00 mm
- net I2C-3_DA: track 54.8 -> 0.00 mm, vias 2 -> 0
- net D8_NEOPIX: track 24.6 -> 0.00 mm, vias 3 -> 0
- net D14: track 20.1 -> 44.5 mm, vias 2 -> 5
- net BACKUP2: track 22.3 -> 0.00 mm, vias 2 -> 0
- net 3.3V: track 79.9 -> 74.6 mm, vias 51 -> 48
- net SDIO_CMD: track 35.2 -> 30.5 mm
- net SDIO_CLK: track 36.5 -> 32.3 mm
- net GND: track 186.2 -> 183.8 mm, vias 65 -> 62
- net SDIO_D1: track 30.9 -> 28.9 mm
- net D13: track 45.5 -> 44.1 mm
- net VISION_TX: track 29.8 -> 28.8 mm
- net VISION_RX: track 27.8 -> 26.8 mm
