File: Robomaster-Controller-Board-v4.0/Kevin's Version/RMCB4.sch (EAGLE design)
At the start: 98 parts, among them Q1 3.1A/30V/105mΩ, SW1 EG1319, U2 AP2112-3.3, X4 32.768, Y2 12mhz

Commit message: Updated Schematic
Parts:
- removed AUX_GPIO2: S2B-PH-SM4_TB, KevinMade:S2B-PH-SM4_TB
- removed I2C_3, I2C_6: SM04B-GHS-TB(LF)(SN)-, SM04B-GHS-TB_LF__SN_-:SM04B-GHS-TB(LF)(SN)-
- added GPIO_AUX1, GPIO_AUX2: S2B-PH-SM4_TB, KevinMade:S2B-PH-SM4_TB
- renumbered PC1 to PC13
Connections:
- net D10 renamed PB9
- net D9 renamed PB8
- net MISO renamed PB14
- net MOSI renamed PB15
- net SCK renamed PB13
- removed net BACKUP2: AUX_GPIO2.JST2, STM32F405RGTX.PC5/ADC12_IN15
- removed net D8_NEOPIX: NEO.DI, STM32F405RGTX.PC0/ADC123_IN10(5T)
- removed net I2C-3_CL: I2C_3.2, I2C_6.2, RN1C.1, STM32F405RGTX.PA8/TIM1_CH1(5T)
- removed net I2C-3_DA: I2C_3.3, I2C_6.3, RN1D.1, STM32F405RGTX.PC9/TIM3_CH4/TIM8_CH4(5T)
- new net GPIO_AUX1: GPIO_AUX1.JST2, STM32F405RGTX.PC5/ADC12_IN15
- new net GPIO_AUX2: GPIO_AUX2.JST2, STM32F405RGTX.PC4/ADC12_IN14
- new net NEOPIX: NEO.DI, STM32F405RGTX.PA8/TIM1_CH1(5T)
- new net PC13: R12.1, STM32F405RGTX.PC13(5T)
- new net PC6: STM32F405RGTX.PC6/TIM3_CH1/TIM_CH1/USART6_TX(5T)
- new net PC7: STM32F405RGTX.PC7/TIM3_CH2/TIM8_CH2/USART6_RX(5T)
- net 3.3V: no longer I2C_3.1, I2C_6.1, RN1C.2, RN1D.2, STM32F405RGTX.PA10/TIM1_CH3/USART1_RX(5T), STM32F405RGTX.PA9/TIM1_CH2/USART1_TX(5T)
- net D13: no longer R12.1
- net D14: now also STM32F405RGTX.PC0/ADC123_IN10(5T); no longer STM32F405RGTX.PC4/ADC12_IN14
- net GND: now also GPIO_AUX1.JST3, GPIO_AUX2.JST3; no longer AUX_GPIO2.JST3, I2C_3.4, I2C_6.4
- net SDIO_CLK: now also STM32F405RGTX.PC12(5T); no longer STM32F405RGTX.PC7/TIM3_CH2/TIM8_CH2/USART6_RX(5T)
- net SDIO_CMD: now also STM32F405RGTX.PD2/TIM3_ETR(5T); no longer STM32F405RGTX.PC6/TIM3_CH1/TIM_CH1/USART6_TX(5T)
- net SDIO_D1: now also STM32F405RGTX.PC9/TIM3_CH4/TIM8_CH4(5T); no longer STM32F405RGTX.PC13(5T)
- net VISION_RX: now also STM32F405RGTX.PA10/TIM1_CH3/USART1_RX(5T); no longer STM32F405RGTX.PD2/TIM3_ETR(5T)
- net VISION_TX: now also STM32F405RGTX.PA9/TIM1_CH2/USART1_TX(5T); no longer STM32F405RGTX.PC12(5T)
