File: Robomaster-Controller-Board-v4.0/RMCB4.sch (EAGLE design)
At the start: 82 parts, among them J1 XT30PW-M, SW1 EG1319, X4 32.768, Y2 12mhz

Commit message: Thursday Meeting changes to the brd, waiting for final submit
Parts:
- removed AUX_GPIO1: S2B-PH-SM4_TB, KevinMade:S2B-PH-SM4_TB
- removed C27: 22pF, microbuilder:CAP_4PACK1206
- removed C28: 47nF, microbuilder:CAP_4PACK1206
- removed D+1, D-1: TPB1,27, testpad:TPB1,27
- removed PC1_PLED: RED, microbuilder:LED0805_NOOUTLINE
- removed R15, R16: 10K, microbuilder:RESISTOR_4PACK_NO
- removed R3: 10K, microbuilder:RESISTOR_4PACK
- added C10, C7, C9: 10uF, microbuilder:CAP_CERAMIC0603_NO
- added C11, C12, C13, C14, C16, C8: 1uF, microbuilder:CAP_CERAMIC0603_NO
- added C15: 47nF, microbuilder:CAP_CERAMIC0603_NO
- added C17, C24, C25: 22pF, microbuilder:CAP_CERAMIC0603_NO
- added C26: 100nF, microbuilder:CAP_CERAMIC0603_NO
- added CONN1: STEMMA_I2C_QT, microbuilder:STEMMA_I2C_QT
- added D5: MBR054, microbuilder:DIODE-SCHOTTKYSOD-123
- added PC1: (no value), adafruit:LEDCHIPLED_0603
- added Q1: 3.1A/30V/105mΩ, SparkFun-DiscreteSemi:MOSFET_PCH-DMG2307L
- added R19: 100K, rcl:R-US_R0603
- added R20: 10K, rcl:R-US_R0603
- added RELAY4: S2B-PH-SM4_TB, KevinMade:S2B-PH-SM4_TB
- added RN1, RN2: 10k, SparkFun-Resistors:1KOHM-ARRAY(4)-0805_ARV-1/10W-5%
- added SSR4: G3VM-61VY2, SamacSys_Parts:G3VM-61VY2
- added U$31, U$32, U$35, U$37: MOUNTINGHOLE2.5, microbuilder:MOUNTINGHOLE2.5
- added U2: AP2112-3.3, microbuilder:VREG_SOT23-5
- C18, C22: device microbuilder:CAP_CERAMIC0603_NO -> rcl:C-EUC0603
- C19, C20, C21: device microbuilder:CAP_CERAMIC0805-NOOUTLINE -> rcl:C-EUC0603
- C23: device microbuilder:CAP_4PACK1206 -> microbuilder:CAP_CERAMIC0603_NO
- R1, R2: device microbuilder:RESISTOR_4PACK -> rcl:R-US_R0603
- R10, R14, R9: device microbuilder:RESISTOR0805_NOOUTLINE -> rcl:R-US_R0603
- R11: device microbuilder:RESISTOR_4PACK_NO -> rcl:R-US_R0603
- R12, R13, R17, R18, R27: device microbuilder:RESISTOR_0603_NOOUT -> rcl:R-US_R0603
Connections:
- net CANH renamed CAN_P
- net CANL renamed CAN_N
- net CANRX renamed CANRX_N
- net CANTX renamed CANTX_P
- removed net BACKUP1: U$40.PC4/ADC12_IN14
- removed net BAKCUP1: AUX_GPIO1.JST2
- removed net CTS: U1.P0.10
- new net D14: SSR4.A, U$40.PC4/ADC12_IN14
- new net EN: R20.1, U2.EN
- new net N$32: D5.C, Q1.D
- new net RELAY4: RELAY4.JST2, SSR4.D1
- new net VHI: C7.1, Q1.S, R20.2, U2.IN
- net 24V: now also Q1.G, SSR4.D2
- net 3.3V: now also C10.1, C11.1, C12.1, C13.1, C14.1, C16.1, C26.1, C8.1, C9.1, CONN1G$1.V+, R1.2, R2.2, RN1A.2, RN1B.2, RN1C.2, RN1D.2, RN2B.2, RN2C.2, U2.OUT; no longer R15G$4.2, R16G$3.2, R1G$2.1, R1G$4.1, R2G$2.1, R2G$4.1, R3G$2.1, R3G$4.1
- net D+: no longer D+1.TP
- net D-: no longer D-1.TP
- net FLASH_CS: now also R1.1; no longer R15G$4.1
- net FLASH_MOSI: now also R11.1; no longer R11G$4.1
- net GND: now also C10.2, C11.2, C12.2, C13.2, C14.2, C15.2, C16.2, C17.2, C23.2, C24.2, C25.2, C26.2, C7.2, C8.2, C9.2, CONN1G$1.GND, CONN1G$2.MT, CONN1G$3.MT, PC1.C, R11.2, R19.1, RELAY4.JST3, SSR4.K, U1.P0.10, U2.GND; no longer AUX_GPIO1.JST3, C232.2, C233.2, C234.2, C272.2, C281.2, PC1_PLED.C, R11G$4.2
- net I2C-1_CL: now also CONN1G$1.SCL, RN2B.1; no longer R3G$2.2
- net I2C-1_DA: now also CONN1G$1.SDA, RN2C.1; no longer R3G$4.2
- net I2C-2_CL: now also RN1A.1; no longer R1G$2.2
- net I2C-2_DA: now also RN1B.1; no longer R1G$4.2
- net I2C-3_CL: now also RN1C.1; no longer R2G$2.2
- net I2C-3_DA: now also RN1D.1; no longer R2G$4.2
- net N$10: now also C23.1; no longer C233.1
- net N$11: now also C24.1; no longer C232.1
- net N$12: now also C17.1; no longer C272.1
- net N$13: now also PC1.A; no longer PC1_PLED.A
- net N$22: now also C15.1; no longer C281.1
- net N$9: now also C25.1; no longer C234.1
- net SDIO_D3: now also R2.1; no longer R16G$3.1
- net VBUS: now also D5.A, R19.2
Other:
- note added: "CTS"
- note removed: "CAN"
- note removed: "I2C1"
- note removed: "I2S2_SD"
- note removed: "I2S2ext_SD"
- note removed: "SPI1"
- note removed: "SPI2"
- moved on the sheet: C22

Commit message: final -kevin
Parts:
- removed I2C_3, I2C_6: SM04B-GHS-TB(LF)(SN)-, SM04B-GHS-TB_LF__SN_-:SM04B-GHS-TB(LF)(SN)-
- removed R14: 2K, rcl:R-US_R0603
- removed SW1: EG1319, microbuilder:SWITCH_DPDTEG1390
- removed U$31, U$32, U$35, U$37: MOUNTINGHOLE2.5, microbuilder:MOUNTINGHOLE2.5
- added AUX1: S2B-PH-SM4_TB, KevinMade:S2B-PH-SM4_TB
- added DIPSWITCH: 1571983-3, Switches:1571983-3
- added R3: 2K, rcl:R-US_R0603
- C26: device microbuilder:CAP_CERAMIC0603_NO -> rcl:C-USC0603
- C5, C6: device microbuilder:CAP_CERAMIC0805-NOOUTLINE -> rcl:C-USC0603
- renumbered AUX_GPIO2 to AUX2, CONN1 to QWIIC, J1 to 24V, LED2 to NEO, PC1 to PC13, U$40 to STM32F405RGTX, U$6 to AMMO_DETEC
Connections:
- net D10 renamed PB9
- net D9 renamed PB8
- net MISO renamed PB14
- net MOSI renamed PB15
- net SCK renamed PB13
- removed net BACKUP2: AUX2.JST2, STM32F405RGTX.PC5/ADC12_IN15
- removed net D8_NEOPIX: NEO.DI, STM32F405RGTX.PC0/ADC123_IN10(5T)
- removed net I2C-3_CL: I2C_3.2, I2C_6.2, RN1C.1, STM32F405RGTX.PA8/TIM1_CH1(5T)
- removed net I2C-3_DA: I2C_3.3, I2C_6.3, RN1D.1, STM32F405RGTX.PC9/TIM3_CH4/TIM8_CH4(5T)
- removed net N$4: R14.2, SW1.P2
- new net GPIO_AUX1: AUX1.JST2, STM32F405RGTX.PC5/ADC12_IN15
- new net GPIO_AUX2: AUX2.JST2, STM32F405RGTX.PC4/ADC12_IN14
- new net NEOPIX: NEO.DI, STM32F405RGTX.PA8/TIM1_CH1(5T)
- new net PC13: R12.1, STM32F405RGTX.PC13(5T)
- new net PC6: STM32F405RGTX.PC6/TIM3_CH1/TIM_CH1/USART6_TX(5T)
- new net PC7: STM32F405RGTX.PC7/TIM3_CH2/TIM8_CH2/USART6_RX(5T)
- net 3.3V: now also DIPSWITCH.2; no longer I2C_3.1, I2C_6.1, RN1C.2, RN1D.2, STM32F405RGTX.PA10/TIM1_CH3/USART1_RX(5T), STM32F405RGTX.PA9/TIM1_CH2/USART1_TX(5T), SW1.O2
- net D13: no longer R12.1
- net D14: now also STM32F405RGTX.PC0/ADC123_IN10(5T); no longer STM32F405RGTX.PC4/ADC12_IN14
- net GND: now also AUX1.JST3, R3.1; no longer I2C_3.4, I2C_6.4, SW1.S2
- net MODE_3V: now also DIPSWITCH.3, R3.2; no longer R14.1
- net SDIO_CLK: now also STM32F405RGTX.PC12(5T); no longer STM32F405RGTX.PC7/TIM3_CH2/TIM8_CH2/USART6_RX(5T)
- net SDIO_CMD: now also STM32F405RGTX.PD2/TIM3_ETR(5T); no longer STM32F405RGTX.PC6/TIM3_CH1/TIM_CH1/USART6_TX(5T)
- net SDIO_D1: now also STM32F405RGTX.PC9/TIM3_CH4/TIM8_CH4(5T); no longer STM32F405RGTX.PC13(5T)
- net VISION_RX: now also STM32F405RGTX.PA10/TIM1_CH3/USART1_RX(5T); no longer STM32F405RGTX.PD2/TIM3_ETR(5T)
- net VISION_TX: now also STM32F405RGTX.PA9/TIM1_CH2/USART1_TX(5T); no longer STM32F405RGTX.PC12(5T)
Other:
- moved on the sheet: C26, C5, C6, RELAY4, RN1A, RN1B, RN2B, RN2C
